Commit message: update urdf files to spawn only stls

File: ur_description/urdf/ur10.urdf.xacro (robot description, xacro)
@@ -62,5 +62,5 @@
       <visual>
         <geometry>
-          <mesh filename="package://ur_description/meshes/ur10/visual/base.dae"/>
+          <mesh filename="package://ur_description/meshes/ur10/collision/base.stl"/>
         </geometry>
         <material name="LightGrey">
@@ -93,5 +93,5 @@
       <visual>
         <geometry>
-          <mesh filename="package://ur_description/meshes/ur10/visual/shoulder.dae"/>
+          <mesh filename="package://ur_description/meshes/ur10/collision/shoulder.stl"/>
         </geometry>
         <material name="LightGrey">
@@ -124,5 +124,5 @@
       <visual>
         <geometry>
-          <mesh filename="package://ur_description/meshes/ur10/visual/upperarm.dae"/>
+          <mesh filename="package://ur_description/meshes/ur10/collision/upperarm.stl"/>
         </geometry>
         <material name="LightGrey">
@@ -155,5 +155,5 @@
       <visual>
          <geometry>
-          <mesh filename="package://ur_description/meshes/ur10/visual/forearm.dae"/>
+          <mesh filename="package://ur_description/meshes/ur10/collision/forearm.stl"/>
         </geometry>
         <material name="LightGrey">
@@ -186,5 +186,5 @@
       <visual>
         <geometry>
-          <mesh filename="package://ur_description/meshes/ur10/visual/wrist1.dae"/>
+          <mesh filename="package://ur_description/meshes/ur10/collision/wrist1.stl"/>
         </geometry>
         <material name="LightGrey">
@@ -217,5 +217,5 @@
       <visual>
         <geometry>
-          <mesh filename="package://ur_description/meshes/ur10/visual/wrist2.dae"/>
+          <mesh filename="package://ur_description/meshes/ur10/collision/wrist2.stl"/>
         </geometry>
         <material name="LightGrey">
@@ -248,5 +248,5 @@
       <visual>
         <geometry>
-          <mesh filename="package://ur_description/meshes/ur10/visual/wrist3.dae"/>
+          <mesh filename="package://ur_description/meshes/ur10/collision/wrist3.stl"/>
         </geometry>
         <material name="LightGrey">

File: ur_description/urdf/ur3.urdf.xacro (robot description, xacro)
@@ -61,5 +61,5 @@
       <visual>
         <geometry>
-          <mesh filename="package://ur_description/meshes/ur3/visual/base.dae"/>
+          <mesh filename="package://ur_description/meshes/ur3/collision/base.stl"/>
         </geometry>
         <material name="LightGrey">
@@ -92,5 +92,5 @@
       <visual>
         <geometry>
-          <mesh filename="package://ur_description/meshes/ur3/visual/shoulder.dae"/>
+          <mesh filename="package://ur_description/meshes/ur3/collision/shoulder.stl"/>
         </geometry>
         <material name="LightGrey">
@@ -123,5 +123,5 @@
       <visual>
         <geometry>
-          <mesh filename="package://ur_description/meshes/ur3/visual/upperarm.dae"/>
+          <mesh filename="package://ur_description/meshes/ur3/collision/upperarm.stl"/>
         </geometry>
         <material name="LightGrey">
@@ -154,5 +154,5 @@
       <visual>
          <geometry>
-          <mesh filename="package://ur_description/meshes/ur3/visual/forearm.dae"/>
+          <mesh filename="package://ur_description/meshes/ur3/collision/forearm.stl"/>
         </geometry>
         <material name="LightGrey">
@@ -185,5 +185,5 @@
       <visual>
         <geometry>
-          <mesh filename="package://ur_description/meshes/ur3/visual/wrist1.dae"/>
+          <mesh filename="package://ur_description/meshes/ur3/collision/wrist1.stl"/>
         </geometry>
         <material name="LightGrey">
@@ -216,5 +216,5 @@
       <visual>
         <geometry>
-          <mesh filename="package://ur_description/meshes/ur3/visual/wrist2.dae"/>
+          <mesh filename="package://ur_description/meshes/ur3/collision/wrist2.stl"/>
         </geometry>
         <material name="LightGrey">
@@ -247,5 +247,5 @@
       <visual>
         <geometry>
-          <mesh filename="package://ur_description/meshes/ur3/visual/wrist3.dae"/>
+          <mesh filename="package://ur_description/meshes/ur3/collision/wrist3.stl"/>
         </geometry>
         <material name="LightGrey">

File: ur_description/urdf/ur5.urdf.xacro (robot description, xacro)
@@ -77,5 +77,5 @@
       <visual>
         <geometry>
-          <mesh filename="package://ur_description/meshes/ur5/visual/base.dae" />
+          <mesh filename="package://ur_description/meshes/ur5/collision/base.stl" />
         </geometry>
         <material name="LightGrey">
@@ -108,5 +108,5 @@
       <visual>
         <geometry>
-          <mesh filename="package://ur_description/meshes/ur5/visual/shoulder.dae" />
+          <mesh filename="package://ur_description/meshes/ur5/collision/shoulder.stl" />
         </geometry>
         <material name="LightGrey">
@@ -139,5 +139,5 @@
       <visual>
         <geometry>
-          <mesh filename="package://ur_description/meshes/ur5/visual/upperarm.dae" />
+          <mesh filename="package://ur_description/meshes/ur5/collision/upperarm.stl" />
         </geometry>
         <material name="LightGrey">
@@ -170,5 +170,5 @@
       <visual>
         <geometry>
-          <mesh filename="package://ur_description/meshes/ur5/visual/forearm.dae" />
+          <mesh filename="package://ur_description/meshes/ur5/collision/forearm.stl" />
         </geometry>
         <material name="LightGrey">
@@ -201,5 +201,5 @@
       <visual>
         <geometry>
-          <mesh filename="package://ur_description/meshes/ur5/visual/wrist1.dae" />
+          <mesh filename="package://ur_description/meshes/ur5/collision/wrist1.stl" />
         </geometry>
         <material name="LightGrey">
@@ -232,5 +232,5 @@
       <visual>
         <geometry>
-          <mesh filename="package://ur_description/meshes/ur5/visual/wrist2.dae" />
+          <mesh filename="package://ur_description/meshes/ur5/collision/wrist2.stl" />
         </geometry>
         <material name="LightGrey">
@@ -263,5 +263,5 @@
       <visual>
         <geometry>
-          <mesh filename="package://ur_description/meshes/ur5/visual/wrist3.dae" />
+          <mesh filename="package://ur_description/meshes/ur5/collision/wrist3.stl" />
         </geometry>
         <material name="LightGrey">
